Commit message: internal renaming

File: urdf/cam_model.urdf.xacro (robot description, xacro)
@@ -252,10 +252,4 @@
     </sensor>
   </gazebo>
-<!-- <xacro:include filename="$(find my_robot)/my_urdfs/lidar.urdf.xacro"/>
-  <joint name="lidarGlue" type="fixed">
-    <parent link="base_link"/>
-    <child link="laz_base"/>
-    <origin xyz="${width/4} 0 ${height/2}"/>
-  </joint> -->
   <joint name="hokuyo_joint" type="fixed">
     <axis xyz="0 0 1" />
